File: spartan_mk1/_autosave-spartan_mk1.kicad_pcb (KiCad board)
At the start: 4 copper layers, 87 parts, among them J1 USB_B_Micro, J10 Conn_01x02_Female, J11 Conn_01x02_Female, J12 Conn_01x02_Female, J13 Conn_02x05_Odd_Even, J14 Conn_01x02_Female, J15 Conn_01x08_Female, J18 Conn_01x08_Female, J2 Conn_01x02_Female, J3 Conn_01x02_Female, J4 Conn_01x02_Female, J5 Conn_01x02_Female, J6 Conn_01x02_Female, J7 Conn_01x04_Female, J8 Conn_01x03_Female, J9 Conn_01x03_Female, Q1 2N7002, Q2 2N7002, Q3 AO3401A, SW1 SW_SPST, U1 MPU-6050, U2 AT24C256C-SSHL-T, U3 USBLC6-2SC6, U4 STM32F405RGTx, U5 AMS1117-3.3, U6 TPS5430DDA, Y1 X322516MLB4SI

Commit message: updated placement
Parts:
- moved H4 32.9 mm to (110.0, 69.0)
Changed lines of the file:
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@@
   )
   (module MountingHole:MountingHole_3.2mm_M3_Pad_Via (layer F.Cu)
-    (at 140.462 81.534)
+    (at 110 69)
     (descr "Mounting Hole 3.2mm, M3")
     (tags "mounting hole 3.2mm m3")
