File: spartan_mk1/Inputs.sch (KiCad schematic (older format))
At the start: 23 parts, among them J1 USB_B_Micro, J10 Conn_01x02_Female, J11 Conn_01x02_Female, J12 Conn_01x02_Female, J13 Conn_02x05_Odd_Even, J2 Conn_01x03_Female, J3 Conn_01x03_Female, J4 Conn_01x03_Female, J5 Conn_01x03_Female, J6 Conn_01x03_Female, J7 Conn_01x05_Female, J8 Conn_01x03_Female, J9 Conn_01x03_Female, Q1 2N7002, Q2 2N7002, U3 USBLC6-2SC6

Commit message: Footprints added started PCB placement
Parts:
- J1: footprint (none) -> Connector_USB:USB_Micro-B_Molex-105017-0001
- J10, J12: footprint (none) -> Connector_SMD:01x02_1.5mm
- J11: footprint (none) -> Connector_SMD:01x02_3mm
- J13: footprint (none) -> Connector_PinHeader_1.27mm:PinHeader_2x05_P1.27mm_Horizontal
- J2, J3, J4, J5, J6: value Conn_01x03_Female -> Conn_01x02_Female; footprint (none) -> Connector_SMD:01x02_1.5mm; symbol Connector:Conn_01x03_Female -> Connector:Conn_01x02_Female
- J7: value Conn_01x05_Female -> Conn_01x04_Female; footprint (none) -> Connector_JST:JST_SH_BM04B-SRSS-TB_1x04-1MP_P1.00mm_Vertical; symbol Connector:Conn_01x05_Female -> Connector:Conn_01x04_Female
- J8, J9: footprint (none) -> Connector_SMD:01x03_1.5mm
- R10, R6: footprint (none) -> Resistor_SMD:R_0805_2012Metric
- R11, R5, R7, R8, R9: footprint (none) -> Resistor_SMD:R_0402_1005Metric
Connections:
- net GND: no longer J2.3 (Pin_3), J3.3 (Pin_3), J4.3 (Pin_3), J5.3 (Pin_3), J6.3 (Pin_3), J7.4 (Pin_4)
- net SPI_CS: now also J7.4 (Pin_4); no longer J7.5 (Pin_5)
Other:
- note added: "Micro USB input (Molex 105017-0001)\nShield should be connected to ground on host side.\n90 ohm controlled impedance trace\n"
- note removed: "Micro USB input\nShield should be connected to ground on host side.\n90 ohm controlled impedance trace\n"

Commit message: updated placement
Parts:
- J13: footprint Connector_PinHeader_1.27mm:PinHeader_2x05_P1.27mm_Horizontal -> Connector_PinHeader_1.27mm:PinHeader_2x05_P1.27mm_Vertical_SMD
Changed lines of the file:
@@
 F 0 "J13" H 9150 2167 50  0000 C CNN
 F 1 "Conn_02x05_Odd_Even" H 9150 2076 50  0000 C CNN
-F 2 "Connector_PinHeader_1.27mm:PinHeader_2x05_P1.27mm_Horizontal" H 9100 1750 50  0001 C CNN
+F 2 "Connector_PinHeader_1.27mm:PinHeader_2x05_P1.27mm_Vertical_SMD" H 9100 1750 50  0001 C CNN
 F 3 "~" H 9100 1750 50  0001 C CNN
 	1    9100 1750

Commit message: Routing in progress
Parts:
- removed J7: Conn_01x04_Female, Connector_JST:JST_SH_BM04B-SRSS-TB_1x04-1MP_P1.00mm_Vertical, symbol Connector:Conn_01x04_Female
- removed R7, R8: 10k, Resistor_SMD:R_0402_1005Metric, symbol Device:R_Small
Connections:
- net +5V: no longer U3.5 (VBUS)
- net V_USB: now also U3.5 (VBUS)
Other:
- note removed: "SPI"
- note removed: "USB Connection Sensing Divider\n"
- note removed: "USB FB"
Changed lines of the file:
@@
 $Descr A4 11693 8268
 encoding utf-8
-Sheet 3 6
+Sheet 5 6
 Title ""
 Date ""
@@
 Text Notes 1000 3150 0    157  ~ 0
 UART Connections
-Text Notes 4050 3150 0    157  ~ 0
-SPI
-$Comp
-L Connector:Conn_01x04_Female J7
-U 1 1 5FB46CD9
-P 4000 3700
-F 0 "J7" H 3892 4085 50  0000 C CNN
-F 1 "Conn_01x04_Female" H 3892 3994 50  0000 C CNN
-F 2 "Connector_JST:JST_SH_BM04B-SRSS-TB_1x04-1MP_P1.00mm_Vertical" H 4000 3700 50  0001 C CNN
-F 3 "~" H 4000 3700 50  0001 C CNN
-	1    4000 3700
-	-1   0    0    -1
-$EndComp
 Wire Notes Line
 	1050 3200 3100 3200
-Wire Notes Line
-	3550 3200 3550 4250
 Text HLabel 1800 4200 2    50   Input ~ 0
 UART2_TX
@@
 Text HLabel 1800 5700 2    50   Input ~ 0
 UART4_RX
-Text HLabel 4250 3600 2    50   Input ~ 0
-SPI_SCK
-Text HLabel 4250 3700 2    50   Input ~ 0
-SPI_MOSI
-Text HLabel 4250 3800 2    50   Input ~ 0
-SPI_MISO
-Text HLabel 4250 3900 2    50   Input ~ 0
-SPI_CS
-Wire Wire Line
-	4250 3600 4200 3600
-Wire Wire Line
-	4250 3700 4200 3700
-Wire Wire Line
-	4250 3800 4200 3800
-Wire Wire Line
-	4250 3900 4200 3900
-Wire Notes Line
-	3550 3200 5100 3200
-Wire Notes Line
-	5100 3200 5100 4250
-Wire Notes Line
-	3550 4250 5100 4250
 Text Notes 3900 4900 0    157  ~ 0
 GPIO
@@
 Wire Notes Line
 	6050 2400 6050 1100
-$Comp
-L power:+5V #PWR017
-U 1 1 5F9DB766
-P 4500 1250
-F 0 "#PWR017" H 4500 1100 50  0001 C CNN
-F 1 "+5V" H 4515 1423 50  0000 C CNN
-F 2 "" H 4500 1250 50  0001 C CNN
-F 3 "" H 4500 1250 50  0001 C CNN
-	1    4500 1250
-	1    0    0    -1
-$EndComp
-Wire Wire Line
-	4500 1250 4500 1300
-Text Notes 5650 3250 0    157  ~ 0
-USB FB
-Text Notes 5650 4450 0    50   ~ 0
-USB Connection Sensing Divider\n
-Wire Notes Line
-	5650 3350 5650 4350
-Wire Notes Line
-	7100 3350 5650 3350
-Wire Notes Line
-	7100 4350 7100 3350
-Wire Notes Line
-	5650 4350 7100 4350
-Text Label 5900 3650 2    50   ~ 0
-Vusb
-Text HLabel 6650 3650 2    50   Input ~ 0
-USB_con
-Wire Wire Line
-	6650 3650 6550 3650
-Wire Wire Line
-	6550 3650 6250 3650
-Connection ~ 6550 3650
-Wire Wire Line
-	6550 3750 6550 3650
-Wire Wire Line
-	6550 3950 6550 4050
-$Comp
-L power:GND #PWR026
-U 1 1 5F97004F
-P 6550 4050
-AR Path="/5F78701C/5F97004F" Ref="#PWR026"  Part="1"
-AR Path="/5F79A745/5F97004F" Ref="#PWR?"  Part="1"
-F 0 "#PWR026" H 6550 3800 50  0001 C CNN
-F 1 "GND" H 6555 3877 50  0000 C CNN
-F 2 "" H 6550 4050 50  0001 C CNN
-F 3 "" H 6550 4050 50  0001 C CNN
-	1    6550 4050
-	1    0    0    -1
-$EndComp
-$Comp
-L Device:R_Small R8
-U 1 1 5F970049
-P 6550 3850
-AR Path="/5F78701C/5F970049" Ref="R8"  Part="1"
-AR Path="/5F79A745/5F970049" Ref="R?"  Part="1"
-F 0 "R8" H 6491 3804 50  0000 R CNN
-F 1 "10k" H 6491 3895 50  0000 R CNN
-F 2 "Resistor_SMD:R_0402_1005Metric" H 6550 3850 50  0001 C CNN
-F 3 "~" H 6550 3850 50  0001 C CNN
-	1    6550 3850
-	-1   0    0    1
-$EndComp
-$Comp
-L Device:R_Small R7
-U 1 1 5F970043
-P 6150 3650
-AR Path="/5F78701C/5F970043" Ref="R7"  Part="1"
-AR Path="/5F79A745/5F970043" Ref="R?"  Part="1"
-F 0 "R7" V 5954 3650 50  0000 C CNN
-F 1 "10k" V 6045 3650 50  0000 C CNN
-F 2 "Resistor_SMD:R_0402_1005Metric" H 6150 3650 50  0001 C CNN
-F 3 "~" H 6150 3650 50  0001 C CNN
-	1    6150 3650
-	0    1    1    0
-$EndComp
 Text HLabel 9450 1550 2    50   Input ~ 0
 SWD_SWDIO
@@
 	5750 5800 5800 5800
 Connection ~ 5800 5800
-Wire Wire Line
-	6050 3650 5900 3650
 Wire Notes Line
 	5250 4900 7650 4900
@@
 Wire Notes Line
 	5250 4900 5250 6450
+Text HLabel 4500 1200 2    50   Input ~ 0
+V_USB
+Wire Wire Line
+	4500 1200 4500 1300
 $EndSCHEMATC

Commit message: Generated gerber files. Positions and BOM assemly files generated
Parts:
- Q1, Q2: LCSC (none) -> C8545; LCSC Part # (none) -> C8545
- R10, R6: LCSC (none) -> C17408; LCSC Part # (none) -> C17408
- R11: LCSC (none) -> C25744; LCSC Part # (none) -> C25744
- R5, R9: LCSC (none) -> C26083; LCSC Part # (none) -> C26083
- U3: LCSC (none) -> C7519; LCSC Part # (none) -> C7519
Changed lines of the file:
@@
 F 2 "Resistor_SMD:R_0402_1005Metric" H 8900 4850 50  0001 C CNN
 F 3 "~" H 8900 4850 50  0001 C CNN
+F 4 "C26083" H 8900 4850 50  0001 C CNN "LCSC Part #"
+F 5 "C26083" H 8900 4850 50  0001 C CNN "LCSC"
 	1    8900 4850
 	1    0    0    -1
@@
 F 2 "Resistor_SMD:R_0402_1005Metric" H 9550 4250 50  0001 C CNN
 F 3 "~" H 9550 4250 50  0001 C CNN
+F 4 "C25744" H 9550 4250 50  0001 C CNN "LCSC Part #"
+F 5 "C25744" H 9550 4250 50  0001 C CNN "LCSC"
 	1    9550 4250
 	1    0    0    -1
@@
 F 2 "Resistor_SMD:R_0805_2012Metric" H 9100 4700 50  0001 C CNN
 F 3 "~" H 9100 4700 50  0001 C CNN
+F 4 "C17408" H 9100 4700 50  0001 C CNN "LCSC Part #"
+F 5 "C17408" H 9100 4700 50  0001 C CNN "LCSC"
 	1    9100 4700
 	0    1    1    0
@@
 F 2 "Package_TO_SOT_SMD:SOT-23" H 9650 4625 50  0001 L CIN
 F 3 "https://www.fairchildsemi.com/datasheets/2N/2N7002.pdf" H 9450 4700 50  0001 L CNN
+F 4 "C8545" H 9450 4700 50  0001 C CNN "LCSC Part #"
+F 5 "C8545" H 9450 4700 50  0001 C CNN "LCSC"
 	1    9450 4700
 	1    0    0    -1
@@
 F 2 "Package_TO_SOT_SMD:SOT-23-6" H 4500 1200 50  0001 C CNN
 F 3 "https://www.st.com/resource/en/datasheet/usblc6-2.pdf" H 4700 2050 50  0001 C CNN
+F 4 "C7519" H 4500 1700 50  0001 C CNN "LCSC Part #"
+F 5 "C7519" H 4500 1700 50  0001 C CNN "LCSC"
 	1    4500 1700
 	1    0    0    -1
@@
 F 2 "Resistor_SMD:R_0402_1005Metric" H 5800 5950 50  0001 C CNN
 F 3 "~" H 5800 5950 50  0001 C CNN
+F 4 "C26083" H 5800 5950 50  0001 C CNN "LCSC Part #"
+F 5 "C26083" H 5800 5950 50  0001 C CNN "LCSC"
 	1    5800 5950
 	1    0    0    -1
@@
 F 2 "Resistor_SMD:R_0805_2012Metric" H 6000 5800 50  0001 C CNN
 F 3 "~" H 6000 5800 50  0001 C CNN
+F 4 "C17408" H 6000 5800 50  0001 C CNN "LCSC Part #"
+F 5 "C17408" H 6000 5800 50  0001 C CNN "LCSC"
 	1    6000 5800
 	0    1    1    0
@@
 F 2 "Package_TO_SOT_SMD:SOT-23" H 6550 5725 50  0001 L CIN
 F 3 "https://www.fairchildsemi.com/datasheets/2N/2N7002.pdf" H 6350 5800 50  0001 L CNN
+F 4 "C8545" H 6350 5800 50  0001 C CNN "LCSC Part #"
+F 5 "C8545" H 6350 5800 50  0001 C CNN "LCSC"
 	1    6350 5800
 	1    0    0    -1
